Commit message: Minor fix on fake_gripper joint bound

File: urdf/fake_gripper.urdf.xacro (robot description, xacro)
@@ -21,5 +21,5 @@
             <axis xyz="0 1 0"/>
             <origin xyz="0 0 0" rpy="0 0 0"/>
-            <limit lower="0" upper="1.4" effort="1" velocity="1"/>
+            <limit lower="-.1" upper="1.4" effort="1" velocity="1"/>
             <!-- <dynamics damping="0.5"/> -->
             <xacro:unless value="${is_master}">
