Commit message: Follow new prl_u5_robot standard for SRDF -- Remove fake gripper controller

File: urdf/cylinder_tool.srdf.xacro (robot description, xacro)
@@ -1,15 +1,13 @@
 <?xml version="1.0" encoding="UTF-8"?>
 <robot xmlns:xacro="http://wiki.ros.org/xacro">
-    <xacro:include filename="$(find prl_ur5_robot_configuration)/urdf/fake_gripper.srdf.xacro"/>
-    <xacro:macro name="cylinder_tool_group" params="prefix">
-        <xacro:fake_gripper_group prefix="${prefix}"/>
-        <link name="${prefix}_base"/>
-        <link name="${prefix}_body"/>
+    <xacro:macro name="cylinder_tool_group_define" params="group_name prefix">
+        <group name="${group_name}">
+            <link name="${prefix}_base"/>
+            <link name="${prefix}_body"/>
+        </group>
     </xacro:macro>
     <xacro:macro name="cylinder_tool_autocol" params="prefix">
-        <xacro:fake_gripper_autocol prefix="${prefix}"/>
     </xacro:macro>
     <xacro:macro name="cylinder_tool_col_with" params="prefix link">
-        <xacro:fake_gripper_col_with prefix="${prefix}" link="${link}"/>
         <disable_collisions link1="${prefix}_body" link2="${link}" reason="Never"/>
     </xacro:macro>

File: urdf/cylinder_tool.urdf.xacro (robot description, xacro)
@@ -47,7 +47,4 @@
         <origin xyz="0 0 0.154" rpy="0 0 0"/>
       </joint>
-      <!-- Create a 'fake' actuated gripper so Moveit don't throw error because it can't find the gripper links/joints/controller from Gazebo -->
-      <xacro:include filename="$(find prl_ur5_robot_configuration)/urdf/fake_gripper.urdf.xacro"/>
-      <xacro:fake_gripper_actuation prefix="${prefix}" palm="${prefix}_body"/>
   </xacro:macro>
 </robot>

File: urdf/no_gripper.srdf.xacro (robot description, xacro)
@@ -1,14 +1,12 @@
 <?xml version="1.0" encoding="UTF-8"?>
 <robot xmlns:xacro="http://wiki.ros.org/xacro">
-    <xacro:include filename="$(find prl_ur5_robot_configuration)/urdf/fake_gripper.srdf.xacro"/>
-    <xacro:macro name="no_gripper_group" params="prefix">
-        <xacro:fake_gripper_group prefix="${prefix}"/>
-        <link name="${prefix}_base"/>
+    <xacro:macro name="no_gripper_group_define" params="group_name prefix">
+        <group name="${group_name}">
+            <link name="${prefix}_base"/>
+        </group>
     </xacro:macro>
     <xacro:macro name="no_gripper_autocol" params="prefix">
-        <xacro:fake_gripper_autocol prefix="${prefix}"/>
     </xacro:macro>
     <xacro:macro name="no_gripper_col_with" params="prefix link">
-        <xacro:fake_gripper_col_with prefix="${prefix}" link="${link}"/>
     </xacro:macro>
 </robot>

File: urdf/no_gripper.urdf.xacro (robot description, xacro)
@@ -2,28 +2,25 @@
 <robot xmlns:xacro="http://wiki.ros.org/xacro">
   <xacro:macro name="no_gripper" params="parent *origin prefix transmission_hw_interface">
-      <link name="${prefix}_base">
-        <inertial>
-        <!-- Add a non-null mass otherwise Gazebo don't load link -->
-          <mass value="0.001" />
-          <inertia  ixx="0.0" ixy="0.0" ixz="0.0"
-                    iyy="0.0" iyz="0.0"
-                    izz="0.0" />
-        </inertial>
-    </link>
-      <joint name="${prefix}_base_joint" type="fixed">
-        <parent link="${parent}"/>
-        <child link = "${prefix}_base"/>
-        <xacro:insert_block name="origin"/>
-      </joint>
-      <!-- grasp frame -->
-      <link name="${prefix}_grasp_frame"/>
-      <joint name="${prefix}_grasp_frame_joint" type="fixed">
-        <parent link="${prefix}_base"/>
-        <child link = "${prefix}_grasp_frame"/>
-        <origin xyz="0 0 0" rpy="0 0 0"/>
-      </joint>
-      <!-- Create a 'fake' actuated gripper so Moveit don't throw error because it can't find the gripper links/joints/controller from Gazebo -->
-      <xacro:include filename="$(find prl_ur5_robot_configuration)/urdf/fake_gripper.urdf.xacro"/>
-      <xacro:fake_gripper_actuation prefix="${prefix}" palm="${prefix}_base"/>
+  <link name="${prefix}_base">
+          <inertial>
+          <!-- Add a non-null mass otherwise Gazebo don't load link -->
+            <mass value="0.001" />
+            <inertia  ixx="0.0" ixy="0.0" ixz="0.0"
+                      iyy="0.0" iyz="0.0"
+                      izz="0.0" />
+          </inertial>
+      </link>
+        <joint name="${prefix}_base_joint" type="fixed">
+          <parent link="${parent}"/>
+          <child link = "${prefix}_base"/>
+          <xacro:insert_block name="origin"/>
+        </joint>
+        <!-- grasp frame -->
+        <link name="${prefix}_grasp_frame"/>
+        <joint name="${prefix}_grasp_frame_joint" type="fixed">
+          <parent link="${prefix}_base"/>
+          <child link = "${prefix}_grasp_frame"/>
+          <origin xyz="0 0 0" rpy="0 0 0"/>
+        </joint>
   </xacro:macro>
 </robot>
