Commit message: Make cylinder 'gripper' collision meshes convex

File: urdf/cylinder_tool.urdf.xacro (robot description, xacro)
@@ -12,5 +12,5 @@
         <visual>
           <geometry>
-            <mesh filename="package://prl_ur5_robot_configuration/urdf/models/cylinder_tool.stl" scale="0.001 0.001 0.001"/>
+            <mesh filename="package://prl_ur5_robot_configuration/urdf/models/cylinder_tool_visual.stl"/>
           </geometry>
           <material name="Grey">
@@ -20,5 +20,10 @@
         <collision>
           <geometry>
-            <mesh filename="package://prl_ur5_robot_configuration/urdf/models/cylinder_tool.stl" scale="0.001 0.001 0.001"/>
+            <mesh filename="package://prl_ur5_robot_configuration/urdf/models/cylinder_tool_collision_body.stl"/>
+          </geometry>
+        </collision>
+        <collision>
+          <geometry>
+            <mesh filename="package://prl_ur5_robot_configuration/urdf/models/cylinder_tool_collision_base.stl"/>
           </geometry>
         </collision>

Commit message: update camera config

File: urdf/cylinder_tool.urdf.xacro (robot description, xacro)
@@ -12,5 +12,5 @@
         <visual>
           <geometry>
-            <mesh filename="package://prl_ur5_robot_configuration/urdf/models/cylinder_tool_visual.stl"/>
+            <mesh filename="file://$(find prl_ur5_robot_configuration)/urdf/models/cylinder_tool_visual.stl"/>
           </geometry>
           <material name="Grey">
@@ -20,10 +20,10 @@
         <collision>
           <geometry>
-            <mesh filename="package://prl_ur5_robot_configuration/urdf/models/cylinder_tool_collision_body.stl"/>
+            <mesh filename="file://$(find prl_ur5_robot_configuration)/urdf/models/cylinder_tool_collision_body.stl"/>
           </geometry>
         </collision>
         <collision>
           <geometry>
-            <mesh filename="package://prl_ur5_robot_configuration/urdf/models/cylinder_tool_collision_base.stl"/>
+            <mesh filename="file://$(find prl_ur5_robot_configuration)/urdf/models/cylinder_tool_collision_base.stl"/>
           </geometry>
         </collision>
